File: hardware/STM32_100pin_Variant/sc_uc.kicad_sch (KiCad schematic)
At the start: 29 parts, among them J6 , U10 STM32L4S7VITx, U11 ATA6561-GAQW-N, Y4 Crystal_GND24

Commit message: Removed OSC_IN Test Point
Test point removed to prevent - --increased capacitance and noise on the high-frequency crystal oscillator line. Can hook up oscilloscope directly to crystal's capacitor when needed.
Parts:
- removed TP8: (no value), TestPoint:TestPoint_Loop_D2.54mm_Drill1.5mm_Beaded, symbol Connector:TestPoint
Changed lines of the file:
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@@
   (junction (at 163.83 19.05) (diameter 0) (color 0 0 0 0)
-  )
-  (junction (at 20.32 67.31) (diameter 0) (color 0 0 0 0)
   )
   (junction (at 205.74 54.61) (diameter 0) (color 0 0 0 0)
@@
     (pin "2")
   )
-  (symbol (lib_id "Connector:TestPoint") (at 20.32 67.31 0) (unit 1)
-    (in_bom yes) (on_board yes)
-    (property "Reference" "TP8" (id 0) (at 17.78 62.23 0)
-      (effects (font (size 1.27 1.27)) (justify left))
-    )
-    (property "Value" " " (id 1) (at 21.7932 66.6242 0)
-      (effects (font (size 1.27 1.27)) (justify left))
-    )
-    (property "Footprint" "TestPoint:TestPoint_Loop_D2.54mm_Drill1.5mm_Beaded" (id 2) (at 25.4 67.31 0)
-      (effects (font (size 1.27 1.27)) hide)
-    )
-    (property "Datasheet" "~" (id 3) (at 25.4 67.31 0)
-      (effects (font (size 1.27 1.27)) hide)
-    )
-    (pin "1")
-  )
   (symbol (lib_id "power:GND") (at 123.19 30.48 0) (unit 1)
