File: hardware/STM32_100pin_Variant/ramn.kicad_sch (KiCad schematic)
At the start: 28 parts, among them J1 USB_C_Micro, J2 Screw_Terminal_01x03

Commit message: Electrical Fix
- Fixed missing VREF+/- connections on ECUs

- Updated version number to V1.1

- Updated Gerbers

- Updated schematic PDF
Other:
- title: RAMN: Resistant Automotive Miniature Network V1.0 -> RAMN 100 Pin Variant
