File: hardware/V1/0_ramn/usb_uc.sch (KiCad schematic (older format))
At the start: 15 parts, among them J3 , U1 ATA6561-GAQW-N, U2 STM32L443CCTx, Y1 NX3225GD-8MHZ-STD-CRA-3

Commit message: Updated schematics to show BOOT0 resistor settings for STM32L5 microcontrollers
Parts:
- R8: value DNM -> 10k
- R9: value 10k -> DNM
- U2: value STM32L443CCTx -> STM32L552/STM32L562
Changed lines of the file:
@@
 Sheet 2 9
 Title "RAMN: Resistant Automotive Miniature Network V1.0"
-Date "2021-06-01"
+Date "2024-02-20"
 Rev "B2L"
-Comp "Copyright (c) 2021 TOYOTA MOTOR CORPORATION. ALL RIGHTS RESERVED."
+Comp "Copyright (c) 2024 TOYOTA MOTOR CORPORATION. ALL RIGHTS RESERVED."
 Comment1 ""
 Comment2 ""
@@
 AR Path="/5D8BFFCE/5D8CC0AC" Ref="U2"  Part="1"
 F 0 "U2" H 9250 2500 50  0000 C CNN
-F 1 "STM32L443CCTx" H 9350 2400 50  0000 C CNN
+F 1 "STM32L552/STM32L562" H 9350 2400 50  0000 C CNN
 F 2 "Package_QFP:LQFP-48_7x7mm_P0.5mm" H 8400 2600 50  0001 R CNN
 F 3 "http://www.st.com/st-web-ui/static/active/en/resource/technical/document/datasheet/DM00254865.pdf" H 8900 4000 50  0001 C CNN
@@
 AR Path="/5D8BFFCE/5FC52C89" Ref="R9"  Part="1"
 F 0 "R9" H 6850 3950 50  0000 C CNN
-F 1 "10k" H 6850 3850 50  0000 C CNN
+F 1 "DNM" H 6850 3850 50  0000 C CNN
 F 2 "Resistor_SMD:R_0603_1608Metric" H 6950 3950 50  0001 C CNN
 F 3 "~" H 6950 3950 50  0001 C CNN
@@
 AR Path="/5D8BFFCE/5FC99F6B" Ref="R8"  Part="1"
 F 0 "R8" H 6800 3550 50  0000 C CNN
-F 1 "DNM" H 6800 3450 50  0000 C CNN
+F 1 "10k" H 6800 3450 50  0000 C CNN
 F 2 "Resistor_SMD:R_0603_1608Metric" H 6950 3550 50  0001 C CNN
 F 3 "~" H 6950 3550 50  0001 C CNN
