File: hardware/V1revC_kiCAD7/0_ramn/LDO.kicad_sch (KiCad schematic)
At the start: 4 parts, among them U11 NCV8163

Commit message: Added revC
Parts:
- renumbered C40 to C21, C41 to C22, D2 to D1, U11 to U6
