File: hardware/V1revC_kiCAD7/0_ramn/ramn.kicad_pcb (KiCad board)
At the start: 2 copper layers, 85.6 x 54 mm, 106 parts, among them J1 USB_C_Micro, J2 Screw_Terminal_01x03, J3 , J4 , J5 , J6 , U1 ATA6561-GAQW-N, U10 NCV8163, U11 NCV8163, U12 NCV8163, U2 STM32L552/STM32L562, U3 ATA6561-GAQW-N, U4 STM32L552/STM32L562, U5 ATA6561-GAQW-N, U6 STM32L552/STM32L562, U7 ATA6561-GAQW-N, U8 STM32L552/STM32L562, U9 NCV8163, Y1 NX3225GD-8MHZ-STD-CRA-3, Y2 NX3225GD-8MHZ-STD-CRA-3, Y3 NX3225GD-8MHZ-STD-CRA-3, Y4 NX3225GD-8MHZ-STD-CRA-3

Commit message: Added revC
Parts:
- added C44: 4.7uF, Capacitor_SMD:C_0603_1608Metric, F.Cu at (55.7, 51.0)
- added C45: 4.7uF, Capacitor_SMD:C_0603_1608Metric, F.Cu at (72.5, 88.6)
- added C46: 4.7uF, Capacitor_SMD:C_0603_1608Metric, F.Cu at (108.7, 88.6)
- added C47: 4.7uF, Capacitor_SMD:C_0603_1608Metric, F.Cu at (90.7, 51.1)
- moved C39 0.70 mm to (88.8, 52.5)
- moved C9 0.63 mm to (53.8, 52.5)
- renumbered BOOT1 to BOOT0, C2 to C1, C11 to C10, C38 to C11, C39 to C12, C12 to C13, C13 to C14, C14 to C15, C15 to C16, C16 to C17, C17 to C18, C18 to C19, C3 to C2, C19 to C20, C40 to C21, C41 to C22, C20 to C23, C21 to C24, C22 to C25, C23 to C26, C24 to C27, C25 to C28, C26 to C29, C4 to C3, C27 to C30, C42 to C31, C43 to C32, C28 to C33, C29 to C34, C30 to C35, C31 to C36, C32 to C37, C33 to C38, C34 to C39, C5 to C4, C35 to C40, C36 to C41, C37 to C42, C1 to C43, C6 to C5, C7 to C6, C8 to C7, C9 to C8, C10 to C9, D2 to D1, D3 to D2, D4 to D3, D1 to D4, R2 to R1, R11 to R10, R12 to R11, R13 to R12, R14 to R13, R15 to R14, R16 to R15, R17 to R16, R1 to R17, R3 to R2, R4 to R3, R5 to R4, R6 to R5, R7 to R6, R8 to R7, R9 to R8, R10 to R9, RX1 to RX, TP2 to TP1, TP1 to TP2, TX1 to TX, U7 to U10, U8 to U11, U9 to U12, U10 to U3, U3 to U4, U4 to U5, U11 to U6, U5 to U7, U6 to U8, U12 to U9
Connections:
- J3 pad 15: /usb_uc/PB11 -> unconnected-(J3-Pin_15-Pad15)
- J4 pad 15: /ECUB/PB11 -> unconnected-(J4-Pin_15-Pad15)
- J5 pad 15: /ECUC/PB11 -> unconnected-(J5-Pin_15-Pad15)
- J6 pad 15: /ECUD/PB11 -> unconnected-(J6-Pin_15-Pad15)
- U11 pad 22: /ECUD/PB11 -> Net-(U11-PB11)
- U2 pad 22: /usb_uc/PB11 -> Net-(U2-PB11)
- U5 pad 22: /ECUB/PB11 -> Net-(U5-PB11)
- U8 pad 22: /ECUC/PB11 -> Net-(U8-PB11)
Routing:
- net /ECUD/PB11: track 11.5 -> 0.00 mm
- net /usb_uc/PB11: track 11.2 -> 0.00 mm
- net /ECUC/PB11: track 8.92 -> 0.00 mm
- net /ECUB/PB11: track 8.92 -> 0.00 mm
- net GND: track 332.8 -> 339.8 mm, vias 121 -> 122
- net +5V: track 304.8 -> 310.4 mm
- net Net-(U2-PB11): track 0.00 -> 2.44 mm
- net Net-(U8-PB11): track 0.00 -> 1.86 mm
- net Net-(U5-PB11): track 0.00 -> 1.83 mm
- net Net-(U11-PB11): track 0.00 -> 1.82 mm
- net /ECUD/3V3_ECU: track 90.1 -> 89.1 mm
Other:
- board text added: "CAN FD BUS"
- board text added: "RAMN V1 rev C2L"
- board text removed: "CAN BUS"
- board text removed: "RAMN V1 rev B2L"
