File: hardware/V1revC_kiCAD7/0_ramn/ramn.kicad_sch (KiCad schematic)
At the start: 27 parts, among them J1 USB_C_Micro, J2 Screw_Terminal_01x03

Commit message: Added revC
Parts:
- renumbered C2 to C1, C3 to C2, C1 to C43, R2 to R1, R1 to R17, R3 to R2, R4 to R3, R5 to R4, R6 to R5, R7 to R6, R8 to R7, TP2 to TP1, TP1 to TP2
Changed lines of the file:
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@@
   (symbol (lib_id "Connector:TestPoint") (at 35.56 63.5 0) (unit 1)
     (in_bom yes) (on_board yes) (dnp no)
-    (property "Reference" "TP1" (at 34.29 58.42 0)
+    (property "Reference" "TP2" (at 34.29 58.42 0)
       (effects (font (size 1.27 1.27)) (justify left))
     )
@@
       (project "ramn"
         (path "/a57c57ad-7d19-43e7-b34c-fd39133eecde"
-          (reference "TP1") (unit 1)
+          (reference "TP2") (unit 1)
         )
       )
@@
   (symbol (lib_id "Device:R_Small_US") (at 41.91 63.5 270) (unit 1)
     (in_bom yes) (on_board yes) (dnp no)
-    (property "Reference" "R2" (at 44.45 62.23 90)
+    (property "Reference" "R1" (at 44.45 62.23 90)
       (effects (font (size 1.27 1.27)))
     )
@@
       (project "ramn"
         (path "/a57c57ad-7d19-43e7-b34c-fd39133eecde"
-          (reference "R2") (unit 1)
+          (reference "R1") (unit 1)
         )
       )
@@
   (symbol (lib_id "Device:R_Small_US") (at 193.04 50.8 270) (unit 1)
     (in_bom yes) (on_board yes) (dnp no)
-    (property "Reference" "R5" (at 193.04 45.72 90)
+    (property "Reference" "R4" (at 193.04 45.72 90)
       (effects (font (size 1.27 1.27)))
     )
@@
       (project "ramn"
         (path "/a57c57ad-7d19-43e7-b34c-fd39133eecde"
+          (reference "R4") (unit 1)
+        )
+      )
+    )
+  )
+  (symbol (lib_id "Device:R_Small_US") (at 193.04 53.34 270) (unit 1)
+    (in_bom yes) (on_board yes) (dnp no)
+    (property "Reference" "R5" (at 193.04 55.88 90)
+      (effects (font (size 1.27 1.27)))
+    )
+    (property "Value" "0R" (at 193.04 58.42 90)
+      (effects (font (size 1.27 1.27)))
+    )
+    (property "Footprint" "Resistor_SMD:R_0603_1608Metric" (at 193.04 53.34 0)
+      (effects (font (size 1.27 1.27)) hide)
+    )
+    (property "Datasheet" "~" (at 193.04 53.34 0)
+      (effects (font (size 1.27 1.27)) hide)
+    )
+    (pin "2")
+    (pin "1")
+    (instances
+      (project "ramn"
+        (path "/a57c57ad-7d19-43e7-b34c-fd39133eecde"
           (reference "R5") (unit 1)
         )
@@
     )
   )
-  (symbol (lib_id "Device:R_Small_US") (at 193.04 53.34 270) (unit 1)
-    (in_bom yes) (on_board yes) (dnp no)
-    (property "Reference" "R6" (at 193.04 55.88 90)
-      (effects (font (size 1.27 1.27)))
-    )
-    (property "Value" "0R" (at 193.04 58.42 90)
-      (effects (font (size 1.27 1.27)))
-    )
-    (property "Footprint" "Resistor_SMD:R_0603_1608Metric" (at 193.04 53.34 0)
-      (effects (font (size 1.27 1.27)) hide)
-    )
-    (property "Datasheet" "~" (at 193.04 53.34 0)
-      (effects (font (size 1.27 1.27)) hide)
-    )
-    (pin "2")
-    (pin "1")
-    (instances
-      (project "ramn"
-        (path "/a57c57ad-7d19-43e7-b34c-fd39133eecde"
-          (reference "R6") (unit 1)
-        )
-      )
-    )
-  )
   (symbol (lib_id "Connector:TestPoint") (at 189.23 50.8 0) (unit 1)
     (in_bom yes) (on_board yes) (dnp no)
@@
   (symbol (lib_id "Device:R_Small_US") (at 68.58 58.42 0) (mirror y) (unit 1)
     (in_bom yes) (on_board yes) (dnp no)
-    (property "Reference" "R4" (at 64.77 57.15 0)
+    (property "Reference" "R3" (at 64.77 57.15 0)
       (effects (font (size 1.27 1.27)) (justify right))
     )
@@
       (project "ramn"
         (path "/a57c57ad-7d19-43e7-b34c-fd39133eecde"
-          (reference "R4") (unit 1)
+          (reference "R3") (unit 1)
         )
       )
@@
   (symbol (lib_id "Device:C_Small") (at 76.2 54.61 90) (unit 1)
     (in_bom yes) (on_board yes) (dnp no)
-    (property "Reference" "C2" (at 77.47 52.07 90)
+    (property "Reference" "C1" (at 77.47 52.07 90)
       (effects (font (size 1.27 1.27)) (justify left))
     )
@@
       (project "ramn"
         (path "/a57c57ad-7d19-43e7-b34c-fd39133eecde"
-          (reference "C2") (unit 1)
+          (reference "C1") (unit 1)
         )
       )
@@
   (symbol (lib_id "Device:R_Small_US") (at 68.58 50.8 0) (mirror y) (unit 1)
     (in_bom yes) (on_board yes) (dnp no)
-    (property "Reference" "R3" (at 64.77 49.53 0)
+    (property "Reference" "R2" (at 64.77 49.53 0)
       (effects (font (size 1.27 1.27)) (justify right))
     )
@@
       (project "ramn"
         (path "/a57c57ad-7d19-43e7-b34c-fd39133eecde"
-          (reference "R3") (unit 1)
+          (reference "R2") (unit 1)
         )
       )
@@
   (symbol (lib_id "Device:R_Small_US") (at 240.03 58.42 0) (unit 1)
     (in_bom yes) (on_board yes) (dnp no)
-    (property "Reference" "R8" (at 237.49 57.15 0)
+    (property "Reference" "R7" (at 237.49 57.15 0)
       (effects (font (size 1.27 1.27)) (justify right))
     )
@@
       (project "ramn"
         (path "/a57c57ad-7d19-43e7-b34c-fd39133eecde"
-          (reference "R8") (unit 1)
+          (reference "R7") (unit 1)
         )
       )
@@
   (symbol (lib_id "Device:C_Small") (at 246.38 54.61 90) (mirror x) (unit 1)
     (in_bom yes) (on_board yes) (dnp no)
-    (property "Reference" "C3" (at 247.65 52.07 90)
+    (property "Reference" "C2" (at 247.65 52.07 90)
       (effects (font (size 1.27 1.27)) (justify left))
     )
@@
       (project "ramn"
         (path "/a57c57ad-7d19-43e7-b34c-fd39133eecde"
-          (reference "C3") (unit 1)
+          (reference "C2") (unit 1)
         )
       )
@@
   (symbol (lib_id "Device:R_Small_US") (at 240.03 50.8 0) (unit 1)
     (in_bom yes) (on_board yes) (dnp no)
-    (property "Reference" "R7" (at 237.49 49.53 0)
+    (property "Reference" "R6" (at 237.49 49.53 0)
       (effects (font (size 1.27 1.27)) (justify right))
     )
@@
       (project "ramn"
         (path "/a57c57ad-7d19-43e7-b34c-fd39133eecde"
-          (reference "R7") (unit 1)
+          (reference "R6") (unit 1)
         )
       )
@@
   (symbol (lib_id "Connector:TestPoint") (at 40.64 90.17 0) (unit 1)
     (in_bom yes) (on_board yes) (dnp no)
-    (property "Reference" "TP2" (at 42.1132 87.1728 0)
+    (property "Reference" "TP1" (at 42.1132 87.1728 0)
       (effects (font (size 1.27 1.27)) (justify left))
     )
@@
       (project "ramn"
         (path "/a57c57ad-7d19-43e7-b34c-fd39133eecde"
-          (reference "TP2") (unit 1)
+          (reference "TP1") (unit 1)
         )
       )
@@
   (symbol (lib_id "Device:R_Small_US") (at 27.94 92.71 90) (unit 1)
     (in_bom yes) (on_board yes) (dnp no)
-    (property "Reference" "R1" (at 26.67 95.25 90)
+    (property "Reference" "R17" (at 26.67 95.25 90)
       (effects (font (size 1.27 1.27)))
     )
@@
       (project "ramn"
         (path "/a57c57ad-7d19-43e7-b34c-fd39133eecde"
-          (reference "R1") (unit 1)
+          (reference "R17") (unit 1)
         )
       )
@@
   (symbol (lib_id "Device:C_Small") (at 27.94 87.63 90) (unit 1)
     (in_bom yes) (on_board yes) (dnp no)
-    (property "Reference" "C1" (at 31.75 82.55 90)
-      (effects (font (size 1.27 1.27)) (justify left))
-    )
-    (property "Value" "100nF" (at 35.56 85.09 90)
+    (property "Reference" "C43" (at 29.21 81.28 90)
+      (effects (font (size 1.27 1.27)) (justify left))
+    )
+    (property "Value" "100nF" (at 30.48 83.82 90)
       (effects (font (size 1.27 1.27)) (justify left))
     )
@@
       (project "ramn"
         (path "/a57c57ad-7d19-43e7-b34c-fd39133eecde"
-          (reference "C1") (unit 1)
-        )
-      )
+          (reference "C43") (unit 1)
+        )
+      )
