File: hardware/V1revC_kiCAD7/0_ramn/sc_uc.kicad_sch (KiCad schematic)
At the start: 20 parts, among them J6 , U7 ATA6561-GAQW-N, U8 STM32L552/STM32L562, Y4 NX3225GD-8MHZ-STD-CRA-3

Commit message: Added revC
Parts:
- added C47: 4.7uF, Capacitor_SMD:C_0603_1608Metric, symbol Device:C_Small
- renumbered C28 to C33, C29 to C34, C30 to C35, C31 to C36, C32 to C37, C33 to C38, C34 to C39, C35 to C40, R15 to R14, R16 to R15, R17 to R16, U7 to U10, U8 to U11
Connections:
- net GND: now also C47.2
- net PB11: no longer names the net of U11.22 (PB11)
- net PB11: now also C47.1; no longer J6.15 (Pin_15)
- no-connect marks 10 -> 11
