File: hardware/V1revC_kiCAD7/0_ramn/usb_uc.kicad_sch (KiCad schematic)
At the start: 15 parts, among them J3 , U1 ATA6561-GAQW-N, U2 STM32L552/STM32L562, Y1 NX3225GD-8MHZ-STD-CRA-3

Commit message: Added revC
Parts:
- added C44: 4.7uF, Capacitor_SMD:C_0603_1608Metric, symbol Device:C_Small
- renumbered BOOT1 to BOOT0, C11 to C10, C4 to C3, C5 to C4, C6 to C5, C7 to C6, C8 to C7, C9 to C8, C10 to C9, R9 to R8, R10 to R9
Connections:
- net GND: now also C44.2
- net PB11: no longer names the net of U2.22 (PB11)
- net PB11: now also C44.1; no longer J3.15 (Pin_15)
- no-connect marks 2 -> 3
