File: hardware/V1revC_kiCAD7/0_ramn/vanilla_uc.kicad_sch (KiCad schematic)
At the start: 14 parts, among them J4 , U3 ATA6561-GAQW-N, U4 STM32L552/STM32L562, Y2 NX3225GD-8MHZ-STD-CRA-3

Commit message: Added revC
Parts:
- added C45: 4.7uF, Capacitor_SMD:C_0603_1608Metric, symbol Device:C_Small
- renumbered C12 to C13, C13 to C14, C14 to C15, C15 to C16, C16 to C17, C17 to C18, C18 to C19, C19 to C20, R11 to R10, R12 to R11, U3 to U4, U4 to U5
Connections:
- net GND: now also C45.2
- net PB11: no longer names the net of U5.22 (PB11)
- net PB11: now also C45.1; no longer J4.15 (Pin_15)
- no-connect marks 10 -> 11
